Commit message: Working ROS connection to UR

File: urdf/ros2_control.xacro (robot description, xacro)
@@ -1,10 +1,13 @@
 <?xml version="1.0" ?>
 <robot xmlns:xacro="http://ros.org/wiki/xacro">
-  <xacro:macro name="snp_ros2_control" params="name prefix sim:=true">
+  <xacro:macro name="ur10e_ros2_control" params="name prefix sim:=false">
     <ros2_control name="${name}" type="system">
       <hardware>
         <xacro:if value="${sim}">
-          <plugin>fake_components/GenericSystem</plugin>
+          <plugin>mock_components/GenericSystem</plugin>
         </xacro:if>
+        <xacro:unless value="${sim}">
+          <plugin>ur_robot_driver/URPositionHardwareInterface</plugin>
+        </xacro:unless>
       </hardware>
       <joint name="${prefix}shoulder_pan_joint">

File: urdf/smw_workcell.xacro (robot description, xacro)
@@ -8,4 +8,5 @@
    <!-- import main macro -->
    <xacro:include filename="$(find ur_description)/urdf/ur_macro.xacro"/>
+  <xacro:include filename="$(find ur_robot_driver)/urdf/ur.ros2_control.xacro"/>
    <!-- possible 'ur_type' values: ur3, ur3e, ur5, ur5e, ur10, ur10e, ur16e, ur20 -->
    <!-- the default value should raise an error in case this was called without defining the type -->
@@ -39,8 +40,9 @@
    <xacro:arg name="simulation_controllers" default="" />
    <xacro:arg name="camera_calibration_file" default="" />
-   <!-- initial position for simulations (Fake Hardware, Gazebo, Ignition) -->
-   <xacro:arg name="initial_positions_file" default="$(find ur_description)/config/initial_positions.yaml"/>
-    <!-- convert to property to use substitution in function -->
-   <xacro:property name="initial_positions_file" default="$(arg initial_positions_file)"/>
+    <xacro:arg name="ur_script_filename" default="$(find ur_client_library)/resources/external_control.urscript"/>
+    <xacro:arg name="ur_output_recipe_filename" default="$(find ur_robot_driver)/resources/rtde_output_recipe.txt"/>
+    <xacro:arg name="ur_input_recipe_filename" default="$(find ur_robot_driver)/resources/rtde_input_recipe.txt"/>
+    <xacro:arg name="use_mock_hardware" default="false" />
+    <xacro:arg name="mock_sensor_commands" default="false" />
     <!-- URDF Materials -->
     <material name="smw_grey">
@@ -63,27 +65,19 @@
       kinematics_parameters_file="$(arg kinematics_params)"
       physical_parameters_file="$(arg physical_params)"
-      visual_parameters_file="$(arg visual_params)"
-      transmission_hw_interface="$(arg transmission_hw_interface)"
-      safety_limits="$(arg safety_limits)"
-      safety_pos_margin="$(arg safety_pos_margin)"
-      safety_k_position="$(arg safety_k_position)"
-      use_fake_hardware="$(arg use_fake_hardware)"
-      fake_sensor_commands="$(arg fake_sensor_commands)"
-      sim_gazebo="$(arg sim_gazebo)"
-      sim_ignition="$(arg sim_ignition)"
-      headless_mode="$(arg headless_mode)"
-      initial_positions="${xacro.load_yaml(initial_positions_file)}"
-      robot_ip="$(arg robot_ip)"
-      script_filename="$(arg script_filename)"
-      output_recipe_filename="$(arg output_recipe_filename)"
-      input_recipe_filename="$(arg input_recipe_filename)"
-      reverse_ip="$(arg reverse_ip)"
-      script_command_port="$(arg script_command_port)"
-      reverse_port="$(arg reverse_port)"
-      script_sender_port="$(arg script_sender_port)"
-      trajectory_port="$(arg trajectory_port)"
-    >
+      visual_parameters_file="$(arg visual_params)"    >
       <origin xyz="0 0 $(arg cart_height)" rpy="0 0 0" />          <!-- position robot in the world -->
     </xacro:ur_robot>
+    <xacro:ur_ros2_control
+      name="$(arg ur_type)"
+      tf_prefix="$(arg tf_prefix)"
+      kinematics_parameters_file="$(arg kinematics_params)"
+      robot_ip="$(arg robot_ip)"
+      script_filename="$(arg ur_script_filename)"
+      output_recipe_filename="$(arg ur_output_recipe_filename)"
+      input_recipe_filename="$(arg ur_input_recipe_filename)"
+      use_mock_hardware="$(arg use_mock_hardware)"
+      mock_sensor_commands="$(arg mock_sensor_commands)"
+      headless_mode="$(arg headless_mode)"
+    />
     <!-- Cart Support -->
     <link name = "cart">
@@ -135,5 +129,5 @@
       <child link="spray_tcp"/>
     </joint>
-  <xacro:property name="camera_calibration_file" default="$(arg camera_calibration_file)"/>
+  <!-- <xacro:property name="camera_calibration_file" default="$(arg camera_calibration_file)"/>
   <xacro:property name="camera_cal" value="${xacro.load_yaml(camera_calibration_file)}" />
   <link name="camera_color_optical_frame"/>
@@ -143,6 +137,6 @@
     <origin xyz="${camera_cal['camera_mount_to_camera_pos']['x']} ${camera_cal['camera_mount_to_camera_pos']['y']} ${camera_cal['camera_mount_to_camera_pos']['z']}"
             rpy="${camera_cal['camera_mount_to_camera_rpy']['x']} ${camera_cal['camera_mount_to_camera_rpy']['y']} ${camera_cal['camera_mount_to_camera_rpy']['z']}" />
-  </joint>
-  <link name="cal_target_frame"/>
+  </joint> -->
+  <!-- <link name="cal_target_frame"/>
   <joint name="target_mount_to_target" type="fixed">
     <parent link="base_link"/>
@@ -150,5 +144,5 @@
     <origin xyz="${camera_cal['target_mount_to_target_pos']['x']} ${camera_cal['target_mount_to_target_pos']['y']} ${camera_cal['target_mount_to_target_pos']['z']}"
             rpy="${camera_cal['target_mount_to_target_rpy']['x']} ${camera_cal['target_mount_to_target_rpy']['y']} ${camera_cal['target_mount_to_target_rpy']['z']}" />
-  </joint>
+  </joint> -->
     <!-- EOAT camera_tcp TCP -->
     <link name="camera_tcp"/>

File: urdf/workcell.xacro (robot description, xacro)
@@ -3,5 +3,5 @@
   <xacro:include filename="$(find ur10e_support)/urdf/smw_workcell.xacro" />
   <xacro:ur10e_macro />
-  <xacro:include filename="$(find ur10e_support)/urdf/ros2_control.xacro"/>
-  <xacro:snp_ros2_control name="SNP ROS2 Control" prefix=""/>
+  <!-- <xacro:include filename="$(find ur10e_support)/urdf/ros2_control.xacro"/> -->
+  <!-- <xacro:ur10e_ros2_control name="UR10e_ROS2_Control" prefix=""/> -->
 </robot>
